File: 2022/HComparator/HComparator/judge.sch (KiCad schematic (older format))
At the start: 7 parts

Commit message: とりあえず全部セーブ。 Judgement まで動いた気がする。
Parts:
- gave numbers to parts that had none: 7
Changed lines of the file:
@@
 	6700 4150 6700 4300
 $Comp
-L 0_OR1Symbols:NMOS_OR1 M?
+L 0_OR1Symbols:NMOS_OR1 M14
 U 1 1 6312D469
 P 6900 4000
-F 0 "M?" H 7144 4091 50  0000 L CNN
+F 0 "M14" H 7144 4091 50  0000 L CNN
 F 1 "NMOS_OR1" H 7144 4000 50  0000 L CNN
 F 2 "" H 6900 4000 50  0001 C CNN
@@
 	6100 4150 6100 4300
 $Comp
-L 0_OR1Symbols:NMOS_OR1 M?
+L 0_OR1Symbols:NMOS_OR1 M13
 U 1 1 6312D475
 P 5900 4000
-F 0 "M?" H 6144 4091 50  0000 L CNN
+F 0 "M13" H 6144 4091 50  0000 L CNN
 F 1 "NMOS_OR1" H 6144 4000 50  0000 L CNN
 F 2 "" H 5900 4000 50  0001 C CNN
@@
 	5150 4750 5350 4750
 $Comp
-L 0_OR1Symbols:NMOS_OR1 M?
+L 0_OR1Symbols:NMOS_OR1 M10
 U 1 1 6312D490
 P 4950 4750
-F 0 "M?" H 5194 4841 50  0000 L CNN
+F 0 "M10" H 5194 4841 50  0000 L CNN
 F 1 "NMOS_OR1" H 5194 4750 50  0000 L CNN
 F 2 "" H 4950 4750 50  0001 C CNN
@@
 	4950 4150 4950 4300
 $Comp
-L 0_OR1Symbols:NMOS_OR1 M?
+L 0_OR1Symbols:NMOS_OR1 M11
 U 1 1 6312D49D
 P 5150 4000
-F 0 "M?" H 5394 4091 50  0000 L CNN
+F 0 "M11" H 5394 4091 50  0000 L CNN
 F 1 "NMOS_OR1" H 5394 4000 50  0000 L CNN
 F 2 "" H 5150 4000 50  0001 C CNN
@@
 	5400 2850 5400 3100
 $Comp
-L 0_OR1Symbols:PMOS_OR1 M?
+L 0_OR1Symbols:PMOS_OR1 M12
 U 1 1 6312D4B0
 P 5200 2700
-F 0 "M?" H 5444 2791 50  0000 L CNN
+F 0 "M12" H 5444 2791 50  0000 L CNN
 F 1 "PMOS_OR1" H 5444 2700 50  0000 L CNN
 F 2 "" H 5200 2700 50  0001 C CNN
@@
 	4350 2100 4350 2800
 $Comp
-L 0_OR1Symbols:NMOS_OR1 M?
+L 0_OR1Symbols:NMOS_OR1 M9
 U 1 1 6312D4C0
 P 4150 4000
-F 0 "M?" H 4394 4091 50  0000 L CNN
+F 0 "M9" H 4394 4091 50  0000 L CNN
 F 1 "NMOS_OR1" H 4394 4000 50  0000 L CNN
 F 2 "" H 4150 4000 50  0001 C CNN
@@
 $EndComp
 $Comp
-L 0_OR1Symbols:PMOS_OR1 M?
+L 0_OR1Symbols:PMOS_OR1 M8
 U 1 1 6312D4C9
 P 4150 3100
-F 0 "M?" H 4394 3191 50  0000 L CNN
+F 0 "M8" H 4394 3191 50  0000 L CNN
 F 1 "PMOS_OR1" H 4394 3100 50  0000 L CNN
 F 2 "" H 4150 3100 50  0001 C CNN
