File: 2022/HComparator/HComparator/output.sch (KiCad schematic (older format))
At the start: 8 parts, among them M15 PMOS_OR1, M16 NMOS_OR1, M17 PMOS_OR1, M18 NMOS_OR1, M19 PMOS_OR1, M20 NMOS_OR1, M21 PMOS_OR1, M22 NMOS_OR1

Commit message: たぶんシミュレーションうまく行った。
Parts:
- M19: Spice_Model PMOS_OR1 l=1u w=2u -> PMOS_OR1 l=1u w=6u
- M21: Spice_Model PMOS_OR1 l=1u w=2u -> PMOS_OR1 l=1u w=17u
Changed lines of the file:
@@
 $Descr A4 11693 8268
 encoding utf-8
-Sheet 4 4
+Sheet 2 4
 Title ""
 Date ""
@@
 F 3 "" H 5600 2950 50  0001 C CNN
 F 4 "M" H 5950 2750 50  0001 L CNN "Spice_Primitive"
-F 5 "PMOS_OR1 l=1u w=2u" H 5844 2859 50  0000 L CNN "Spice_Model"
+F 5 "PMOS_OR1 l=1u w=6u" H 5844 2859 50  0000 L CNN "Spice_Model"
 F 6 "Y" H 5950 2850 50  0001 L CNN "Spice_Netlist_Enabled"
 	1    5600 2950
@@
 F 3 "" H 6950 2950 50  0001 C CNN
 F 4 "M" H 7300 2750 50  0001 L CNN "Spice_Primitive"
-F 5 "PMOS_OR1 l=1u w=2u" H 7194 2859 50  0000 L CNN "Spice_Model"
+F 5 "PMOS_OR1 l=1u w=17u" H 7194 2859 50  0000 L CNN "Spice_Model"
 F 6 "Y" H 7300 2850 50  0001 L CNN "Spice_Netlist_Enabled"
 	1    6950 2950

Commit message: へ〜いとにかくセーブ
Connections:
- wire segments 73 -> 72
Changed lines of the file:
@@
 	4700 5150 5250 5150
 Wire Wire Line
-	5900 5150 5250 5150
+	5900 5150 5350 5150
 Connection ~ 5250 5150
 Wire Wire Line
-	5250 4650 5250 5150
-Wire Wire Line
-	5350 4650 5250 4650
-Wire Wire Line
-	5350 4400 5350 4650
-Wire Wire Line
 	5250 4400 5350 4400
-Connection ~ 5250 4650
-Wire Wire Line
-	5250 4550 5250 4650
 Wire Wire Line
 	4900 4400 5050 4400
@@
 Wire Wire Line
 	7150 3250 7150 3500
+Wire Wire Line
+	5250 4550 5250 5150
+Wire Wire Line
+	5350 4400 5350 5150
+Connection ~ 5350 5150
+Wire Wire Line
+	5350 5150 5250 5150
 $EndSCHEMATC
