File: 2022/HComparator/HComparator/pre-amp.sch (KiCad schematic (older format))
At the start: 7 parts, among them M1 PMOS_OR1, M2 NMOS_OR1, M3 NMOS_OR1, M4 PMOS_OR1, M5 NMOS_OR1, M6 PMOS_OR1, M7 NMOS_OR1

Commit message: バックアップした。
Connections:
- net VSS: now also M3.4 (B), M7.4 (B)
Changed lines of the file:
@@
 $Descr A4 11693 8268
 encoding utf-8
-Sheet 2 4
+Sheet 4 4
 Title ""
 Date ""
@@
 	1    0    0    -1
 $EndComp
-Wire Wire Line
-	2650 2350 2650 2200
 Connection ~ 2650 2700
 Wire Wire Line
-	2650 5100 4650 5100
-Wire Wire Line
-	4900 4500 4900 4650
+	2650 5100 4550 5100
 Wire Wire Line
 	4900 4350 5050 4350
 Wire Wire Line
-	5050 4350 5050 4650
-Wire Wire Line
-	5050 4650 4900 4650
-Connection ~ 4900 4650
-Wire Wire Line
 	2650 2500 2850 2500
-Wire Wire Line
-	2850 2500 2850 2200
-Wire Wire Line
-	2850 2200 2650 2200
-Connection ~ 2650 2200
-Wire Wire Line
-	2650 2200 2650 1900
 Text HLabel 4300 1650 0    50   Input ~ 0
 VDD
@@
 Connection ~ 4650 1900
 Wire Wire Line
-	4650 1900 5500 1900
+	4650 1900 5350 1900
 Wire Wire Line
 	4350 5300 4650 5300
@@
 	4650 5300 4650 5100
 Connection ~ 4650 5100
-Wire Wire Line
-	4650 5100 4900 5100
 $Comp
 L 0_OR1Symbols:NMOS_OR1 M2
@@
 $EndComp
 Wire Wire Line
-	2650 5100 2650 4700
-Wire Wire Line
-	2300 4700 2650 4700
-Connection ~ 2650 4700
-Wire Wire Line
-	2650 4700 2650 4500
-Wire Wire Line
 	5350 2500 5500 2500
 $Comp
@@
 $EndComp
 Wire Wire Line
-	5350 2200 5350 2500
-Wire Wire Line
-	5500 2200 5500 2350
-Wire Wire Line
-	5500 1900 5500 2200
-Connection ~ 5500 2200
-Wire Wire Line
-	5500 2200 5350 2200
-Wire Wire Line
 	5700 2500 5850 2500
 Wire Wire Line
 	2650 4350 2300 4350
-Wire Wire Line
-	2300 4350 2300 4700
-Wire Wire Line
-	4900 4650 4900 5100
 $Comp
 L 0_OR1Symbols:NMOS_OR1 M3
@@
 	3950 4050 4900 4050
 Wire Wire Line
-	3950 3900 5500 3900
+	3950 3900 4550 3900
 Wire Wire Line
 	4900 4050 4900 4200
@@
 Wire Wire Line
 	4150 3000 4300 3000
-Connection ~ 3950 2700
-Wire Wire Line
-	3750 2700 3950 2700
-Wire Wire Line
-	3750 3000 3750 2700
 Wire Wire Line
 	3950 3000 3750 3000
-Wire Wire Line
-	3950 2850 3950 2700
 $Comp
 L 0_OR1Symbols:PMOS_OR1 M4
@@
 	-1   0    0    -1
 $EndComp
-Wire Wire Line
-	2650 1900 3950 1900
-Wire Wire Line
-	3950 1900 3950 2700
 Connection ~ 3950 1900
 Wire Wire Line
@@
 Text HLabel 3550 3900 0    50   Input ~ 0
 VM
+Wire Wire Line
+	2650 1900 2650 2350
+Wire Wire Line
+	2850 2500 2850 1900
+Wire Wire Line
+	2650 1900 2850 1900
+Connection ~ 2850 1900
+Wire Wire Line
+	2850 1900 3750 1900
+Wire Wire Line
+	3950 1900 3950 2850
+Connection ~ 3750 1900
+Wire Wire Line
+	3750 1900 3950 1900
+Wire Wire Line
+	3750 1900 3750 3000
+Wire Wire Line
+	5500 1900 5500 2350
+Wire Wire Line
+	5350 2500 5350 1900
+Connection ~ 5350 1900
+Wire Wire Line
+	5350 1900 5500 1900
+Wire Wire Line
+	2650 5100 2300 5100
+Connection ~ 2650 5100
+Wire Wire Line
+	2300 4350 2300 5100
+Wire Wire Line
+	2650 4500 2650 5100
+Wire Wire Line
+	4650 5100 4900 5100
+Connection ~ 4900 5100
+Wire Wire Line
+	4900 5100 5050 5100
+Wire Wire Line
+	5050 4350 5050 5100
+Wire Wire Line
+	4900 4500 4900 5100
+Wire Wire Line
+	4550 3900 4550 5100
+Connection ~ 4550 3900
+Wire Wire Line
+	4550 3900 5500 3900
+Connection ~ 4550 5100
+Wire Wire Line
+	4550 5100 4650 5100
 $EndSCHEMATC

Commit message: へ〜いとにかくセーブ
Changed lines of the file:
@@
 $Descr A4 11693 8268
 encoding utf-8
-Sheet 4 4
+Sheet 2 4
 Title ""
 Date ""
@@
 Wire Wire Line
 	2650 3900 3100 3900
-Wire Wire Line
-	3550 3900 3750 3900
 Text HLabel 3550 3900 0    50   Input ~ 0
 VM
@@
 Wire Wire Line
 	4550 5100 4650 5100
+Wire Wire Line
+	3750 3900 3550 3900
 $EndSCHEMATC
