File: 2022/HComparator/HComparator/tb/tb.sch (KiCad schematic (older format))
At the start: 3 parts

Commit message: とりあえず TB は通った。
Connections:
- net Sheet631A3B06/VDD renamed Sheet62FFD227/VDD
Changed lines of the file:
@@
 $Descr A4 11693 8268
 encoding utf-8
-Sheet 1 3
+Sheet 1 4
 Title ""
 Date ""
@@
 Wire Wire Line
 	4550 3350 4300 3350
-$Sheet
-S 6900 3050 1550 1700
-U 631A3B07
-F0 "Sheet631A3B06" 50
-F1 "../judge.sch" 50
-F2 "VDD" I L 6900 3250 50
-F3 "Vin1" I L 6900 3550 50
-F4 "Vin2" I L 6900 3750 50
-F5 "VSS" I L 6900 4150 50
-F6 "Vout1" O R 8450 3550 50
-F7 "Vout2" O R 8450 3800 50
-$EndSheet
-Wire Wire Line
-	6550 3550 6900 3550
-Wire Wire Line
-	6550 3750 6900 3750
 Wire Wire Line
 	4300 3350 4300 2650
 Wire Wire Line
-	4300 2650 6750 2650
-Wire Wire Line
 	6750 2650 6750 3250
-Wire Wire Line
-	6750 3250 6900 3250
 Connection ~ 4300 3350
 Wire Wire Line
@@
 	4300 5100 6750 5100
 Wire Wire Line
-	6750 5100 6750 4150
-Wire Wire Line
-	6750 4150 6900 4150
+	6750 5100 6750 4600
 Connection ~ 4300 4650
 Wire Wire Line
 	4300 4650 3700 4650
+Wire Wire Line
+	4300 2650 6750 2650
+Wire Wire Line
+	6750 5100 8700 5100
+Connection ~ 6750 5100
+Connection ~ 6750 2650
+Wire Wire Line
+	6750 2650 8700 2650
+$Sheet
+S 6850 3000 1600 1750
+U 62FFD228
+F0 "Sheet62FFD227" 50
+F1 "../judge.sch" 50
+F2 "VDD" I L 6850 3250 50
+F3 "Vin1" I L 6850 3550 50
+F4 "Vin2" I L 6850 3750 50
+F5 "VSS" I L 6850 4600 50
+F6 "Vout1" O R 8450 3550 50
+F7 "Vout2" O R 8450 3750 50
+$EndSheet
+Wire Wire Line
+	6850 4600 6750 4600
+Wire Wire Line
+	6550 3550 6850 3550
+Wire Wire Line
+	6550 3750 6850 3750
+Wire Wire Line
+	6750 3250 6850 3250
+Wire Wire Line
+	8700 2650 8700 3350
+Wire Wire Line
+	8700 3950 8700 5100
+$Sheet
+S 9100 3050 1550 1700
+U 63071FC2
+F0 "Sheet63071FC1" 50
+F1 "../output.sch" 50
+F2 "VDD" I L 9100 3350 50
+F3 "Vin1" I L 9100 3550 50
+F4 "Vin2" I L 9100 3750 50
+F5 "Vss" I L 9100 3950 50
+F6 "Vout" O R 10650 3650 50
+$EndSheet
+Wire Wire Line
+	8700 3350 9100 3350
+Wire Wire Line
+	8450 3550 9100 3550
+Wire Wire Line
+	8450 3750 9100 3750
+Wire Wire Line
+	8700 3950 9100 3950
 $EndSCHEMATC

Commit message: バックアップした。
Parts:
- removed V2: VDC, symbol Simulation_SPICE:VDC
- added V2: VPWL, symbol Simulation_SPICE:VPWL
- V3: Spice_Model pwl(0 0 1000n 5 2500n 0) -> pwl(0 0 1u 5 2.5u 0 2510n 4.0 2599n 4.0 2600n 1.6 2699n 1.6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
Connections:
- net 0: now also V2.2
- net Sheet6330DAC5/VP: now also V2.1
Other:
- note added: ".tran 1ns 3000ns 0ns1000ns"
- note removed: ".tran 1ns 2500ns 0ns1000ns"
Changed lines of the file:
@@
-$EndComp
-$Comp
-L Simulation_SPICE:VDC V2
-U 1 1 632C52D7
-P 2550 4250
-F 0 "V2" H 2680 4341 50  0000 L CNN
-F 1 "VDC" H 2680 4250 50  0000 L CNN
-F 2 "" H 2550 4250 50  0001 C CNN
-F 3 "~" H 2550 4250 50  0001 C CNN
-F 4 "Y" H 2550 4250 50  0001 L CNN "Spice_Netlist_Enabled"
-F 5 "V" H 2550 4250 50  0001 L CNN "Spice_Primitive"
-F 6 "dc 2.25" H 2680 4159 50  0000 L CNN "Spice_Model"
-	1    2550 4250
-	1    0    0    -1
 $EndComp
 $Comp
@@
 F 4 "Y" H 3200 4250 50  0001 L CNN "Spice_Netlist_Enabled"
 F 5 "V" H 3200 4250 50  0001 L CNN "Spice_Primitive"
-F 6 "pwl(0 0 1000n 5 2500n 0)" H 3330 4159 50  0000 L CNN "Spice_Model"
+F 6 "pwl(0 0 1u 5 2.5u 0  2510n 4.0 2599n 4.0 2600n 1.6 2699n 1.6 2700n 4)" H 3350 4550 50  0000 L CNN "Spice_Model"
 	1    3200 4250
 	1    0    0    -1
@@
 .include /home/ryos/Project/MakeLSI/MakeLSI/2022/HComparator/HComparator/tb/16PTS/mos_PTS06.lib
 Text Notes 2150 1950 0    50   ~ 0
-.tran 1ns 2500ns  0ns1000ns
+.tran 1ns 3000ns  0ns1000ns
 Connection ~ 3700 4650
 Wire Wire Line
@@
 F7 "VM" I L 4550 4050 50
 $EndSheet
+$Comp
+L Simulation_SPICE:VPWL V2
+U 1 1 62FD6CCD
+P 2550 4250
+F 0 "V2" H 2680 4341 50  0000 L CNN
+F 1 "VPWL" H 2680 4250 50  0000 L CNN
+F 2 "" H 2550 4250 50  0001 C CNN
+F 3 "~" H 2550 4250 50  0001 C CNN
+F 4 "Y" H 2550 4250 50  0001 L CNN "Spice_Netlist_Enabled"
+F 5 "V" H 2550 4250 50  0001 L CNN "Spice_Primitive"
+F 6 "pwl(0 0 100n 2.25 2500n 2.25 2510n 1.6 2600n 1.6 2601n 4.0 2700n 4.0 2701n 1.6 )" H 2680 4159 50  0000 L CNN "Spice_Model"
+	1    2550 4250
+	1    0    0    -1
+$EndComp
 $EndSCHEMATC
