File: 2022/HComparator/KiCad/output.sch (KiCad schematic (older format))
At the start: 8 parts, among them M15 PMOS_OR1, M16 NMOS_OR1, M17 PMOS_OR1, M18 NMOS_OR1, M19 PMOS_OR1, M20 NMOS_OR1, M21 PMOS_OR1, M22 NMOS_OR1

Commit message: KiCad の分割した回路図でも LVS が通るようになった。 シート名称にブランクを入れてはいけない。
Parts:
- M19: Spice_Model PMOS_OR1 l=1u w=6u -> PMOS_OR1 l=1u w=2u
- M21: Spice_Model PMOS_OR1 l=1u w=17u -> PMOS_OR1 l=1u w=6u
Changed lines of the file:
@@
 F 3 "" H 5600 2950 50  0001 C CNN
 F 4 "M" H 5950 2750 50  0001 L CNN "Spice_Primitive"
-F 5 "PMOS_OR1 l=1u w=6u" H 5844 2859 50  0000 L CNN "Spice_Model"
+F 5 "PMOS_OR1 l=1u w=2u" H 5844 2859 50  0000 L CNN "Spice_Model"
 F 6 "Y" H 5950 2850 50  0001 L CNN "Spice_Netlist_Enabled"
 	1    5600 2950
@@
 F 3 "" H 6950 2950 50  0001 C CNN
 F 4 "M" H 7300 2750 50  0001 L CNN "Spice_Primitive"
-F 5 "PMOS_OR1 l=1u w=17u" H 7194 2859 50  0000 L CNN "Spice_Model"
+F 5 "PMOS_OR1 l=1u w=6u" H 7194 2859 50  0000 L CNN "Spice_Model"
 F 6 "Y" H 7300 2850 50  0001 L CNN "Spice_Netlist_Enabled"
 	1    6950 2950
