File: 2023/VCO/KiCad7/VCO.kicad_sch (KiCad schematic)
At the start: 26 parts, among them M27 NMOS_OR1, M28 NMOS_OR1, M29 NMOS_OR1, M30 PMOS_OR1, M31 NMOS_OR1, M32 PMOS_OR1, M33 NMOS_OR1, M34 NMOS_OR1, M35 PMOS_OR1, M36 NMOS_OR1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

Commit message: add TB
Parts:
- added M1, M2, M3, M4: PMOS_OR1, symbol OR1Symbols:PMOS_OR1
Connections:
- net OUT: now also M3.1 (D), M4.4 (B); no longer M31.2 (G), M51.1 (D), M52.1 (D)
- net VDD: now also M1.3 (S), M1.4 (B), M3.3 (S), M3.4 (B)
- new net: M1.1 (D), M2.3 (S), M3.2 (G), M4.2 (G)
- new net: M1.2 (G), M2.1 (D), M2.2 (G), M2.4 (B), M31.2 (G), M4.1 (D), M51.1 (D), M52.1 (D)
Other:
- moved on the sheet: M27, M28, M29, M30, M31, M32, M33, M34, M35, M36, M37, M38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

Commit message: TB もとに戻す。
Parts:
- removed M1, M2, M3, M4: PMOS_OR1, symbol OR1Symbols:PMOS_OR1
Connections:
- net OUT: now also M31.2 (G), M51.1 (D), M52.1 (D)
